Commit message: Basic parameters for pick and place

File: turtlebot_arm_description/urdf/pincher_arm.urdf (robot description, URDF)
Before this commit: robot turtlebot_arm, 24 links, 23 joints
Joints:
- joint arm_elbow_flex_joint: limit lower=-2.617 upper=2.617 effort=30 velocity=1.571 -> lower=-2.42 upper=2.38 effort=30 velocity=1.571
- joint arm_shoulder_lift_joint: limit lower=-2.617 upper=2.617 effort=30 velocity=1.571 -> lower=-2.2 upper=2.16 effort=30 velocity=1.571
- joint arm_wrist_flex_joint: limit lower=-1.745 upper=1.745 effort=30 velocity=1.571 -> lower=-1.72 upper=1.68 effort=30 velocity=1.571
- joint gripper_joint: limit lower=0.002 upper=0.031 effort=30 velocity=0.5 -> lower=0.000 upper=0.0315 effort=30 velocity=0.5

File: turtlebot_arm_description/urdf/pincher_gripper.xacro (robot description, xacro)
@@ -16,5 +16,5 @@
       <origin xyz="0 0 0" rpy="0 0 0"/>
       <axis xyz="1 0 0"/>
-      <limit effort="30" velocity="0.5" lower="0.002" upper="0.031"/>
+      <limit effort="30" velocity="0.5" lower="0.0005" upper="0.0315"/>
       <parent link="gripper_servo_link"/>
       <child link="gripper_active_link"/>

Commit message: Make both parts of the pincher move using a mimic joint

File: turtlebot_arm_description/urdf/pincher_arm.urdf (robot description, URDF)
Before this commit: robot turtlebot_arm, 24 links, 23 joints
Joints:
- joint gripper2_joint: axis (none) -> 1 0 0; limit (none) -> lower=0.0005 upper=0.0155 effort=30 velocity=0.5; mimic (none) -> joint=gripper_joint multiplier=-1 offset=0; origin (none) -> xyz=0 0 0 rpy=0 0 0; type fixed -> prismatic
- joint gripper_finger_base_joint: origin xyz=0.01  0.038 0 rpy=1.570795 -3.14159 1.570795 -> xyz=0.0175  0.038 0 rpy=1.570795 -3.14159 1.570795
- joint gripper_joint: limit lower=0.000 upper=0.0315 effort=30 velocity=0.5 -> lower=0.0005 upper=0.0155 effort=30 velocity=0.5

File: turtlebot_arm_description/urdf/pincher_gripper.xacro (robot description, xacro)
@@ -10,5 +10,5 @@
     </dynamixel_AX12_fixed>
      <gripper_finger_base parent="gripper_servo_link" name="gripper_finger_base" color="${color}">
-      <origin xyz="0.01  ${AX12_WIDTH} 0" rpy="${M_PI/2} ${-M_PI} ${M_PI/2}"/>
+      <origin xyz="0.0175  ${AX12_WIDTH} 0" rpy="${M_PI/2} ${-M_PI} ${M_PI/2}"/>
     </gripper_finger_base>
      <!-- Finger 1 -->
@@ -16,30 +16,29 @@
       <origin xyz="0 0 0" rpy="0 0 0"/>
       <axis xyz="1 0 0"/>
-      <limit effort="30" velocity="0.5" lower="0.0005" upper="0.0315"/>
+      <limit effort="30" velocity="0.5" lower="0.0005" upper="0.0155"/>
       <parent link="gripper_servo_link"/>
       <child link="gripper_active_link"/>
     </joint>
     <pincher_gripper name="gripper_active" color="${color}" >
-      <origin xyz="-0.02 0.023 0" rpy="${-M_PI/2} 0 0"/>
+      <origin xyz="0 0.023 0" rpy="${-M_PI/2} 0 0"/>
     </pincher_gripper>
     <!-- Finger 2 -->
     <!-- Note: currently static but should be a Mimic of Finger 1 -->
-    <joint name="gripper2_joint" type="fixed">
+ <!--   <joint name="gripper2_joint" type="fixed">
       <parent link="gripper_servo_link"/>
       <child link="gripper_active2_link"/>
-    </joint>
+    </joint>   -->
     <pincher_gripper name="gripper_active2" color="${color}" >
-      <origin xyz="-0.02 0.023 0" rpy="${-M_PI/2} ${M_PI} 0"/>
+      <origin xyz="0 0.023 0" rpy="${-M_PI/2} ${M_PI} 0"/>
     </pincher_gripper>
     <!-- Using Mimic -->
     <!-- gripper 2 joint -->
-    <!--  ### Mimic would be better but causes Missing Joint error in Moveit
       <joint name="gripper2_joint" type="prismatic">
       <origin xyz="0 0 0" rpy="0 0 0"/>
-      <axis xyz="0 0 1"/>
-      <limit effort="30" velocity="0.5" lower="0.002" upper="0.031"/>
+      <axis xyz="1 0 0"/>
+      <limit effort="30" velocity="0.5" lower="0.0005" upper="0.0155"/>
       <parent link="gripper_servo_link"/>
       <child link="gripper_active2_link"/>
-      <mimic joint="gripper_joint" multiplier="-.5"  offset = "0"/>
-    </joint-->
+      <mimic joint="gripper_joint" multiplier="-1" offset = "0"/>
+    </joint>
 </robot>

Commit message: Redo limits to allow the pick and place gripper demo to work again
Looks like if move group commander is used on the gripper, the values need
to be doubled or halved, right now it will always think it has failed though
in reality the gripper will reach the intended pose.

This also might cause trouble down the line, as the joint limits are double
what the gripper can reach right now.  Need to look into the commander further
to see why this is happening

File: turtlebot_arm_description/urdf/pincher_arm.urdf (robot description, URDF)
Before this commit: robot turtlebot_arm, 24 links, 23 joints
Joints:
- joint gripper2_joint: limit lower=0.0005 upper=0.0155 effort=30 velocity=0.5 -> lower=-0.031 upper=-0.0005 effort=30 velocity=0.5
- joint gripper_joint: limit lower=0.0005 upper=0.0155 effort=30 velocity=0.5 -> lower=0.0005 upper=0.031 effort=30 velocity=0.5

File: turtlebot_arm_description/urdf/pincher_gripper.xacro (robot description, xacro)
@@ -16,5 +16,5 @@
       <origin xyz="0 0 0" rpy="0 0 0"/>
       <axis xyz="1 0 0"/>
-      <limit effort="30" velocity="0.5" lower="0.0005" upper="0.0155"/>
+      <limit effort="30" velocity="0.5" lower="0.0005" upper="0.031"/>
       <parent link="gripper_servo_link"/>
       <child link="gripper_active_link"/>
@@ -37,5 +37,5 @@
       <origin xyz="0 0 0" rpy="0 0 0"/>
       <axis xyz="1 0 0"/>
-      <limit effort="30" velocity="0.5" lower="0.0005" upper="0.0155"/>
+      <limit effort="30" velocity="0.5" lower="-0.031" upper="-0.0005"/>
       <parent link="gripper_servo_link"/>
       <child link="gripper_active2_link"/>
